Commit message: update urdf files to match current hpp-ipa naming convention

File: urdf/door.urdf.xacro (robot description, xacro)
@@ -11,5 +11,5 @@
                 <origin xyz="0 0 0" rpy="0 0 0" />
                 <geometry>
-                    <mesh filename="package://hpp-dlr-ipa/meshes/Door_m.STL"/>
+                    <mesh filename="package://hpp-ipa/meshes/Door_m.STL"/>
                 </geometry>
                 <material name="greyish">
@@ -20,5 +20,5 @@
                 <origin xyz="0 0 0" rpy="0 0 0" />
                 <geometry>
-                    <mesh filename="package://hpp-dlr-ipa/meshes/Door_m.STL"/>
+                    <mesh filename="package://hpp-ipa/meshes/Door_m.STL"/>
                 </geometry>
             </collision>

File: urdf/platform.urdf.xacro (robot description, xacro)
@@ -18,5 +18,5 @@
                 <origin xyz="0 0 0" rpy="0 0 0" />
                 <geometry>
-                    <mesh filename="package://hpp-dlr-ipa/meshes/Mobile_Platform_Shell_m.STL"/>
+                    <mesh filename="package://hpp-ipa/meshes/Mobile_Platform_Shell_m.STL"/>
                 </geometry>
                 <material name="greyish">
@@ -27,5 +27,5 @@
                 <origin xyz="0 0 0" rpy="0 0 0" />
                 <geometry>
-                    <mesh filename="package://hpp-dlr-ipa/meshes/Mobile_Platform_Shell_m.STL"/>
+                    <mesh filename="package://hpp-ipa/meshes/Mobile_Platform_Shell_m.STL"/>
                 </geometry>
             </collision>

File: urdf/tool_changer.urdf.xacro (robot description, xacro)
@@ -17,5 +17,5 @@
                 <origin xyz="0 0 -0.0742" rpy="0 0 0" />
                 <geometry>
-                    <mesh filename="package://hpp-dlr-ipa/meshes/Tools_to_Tool_Changer_m.STL"/>
+                    <mesh filename="package://hpp-ipa/meshes/Tools_to_Tool_Changer_m.STL"/>
                 </geometry>
                 <material name="greyish">
@@ -26,5 +26,5 @@
                 <origin xyz="0 0 -0.0742" rpy="0 0 0" />
                 <geometry>
-                    <mesh filename="package://hpp-dlr-ipa/meshes/Tools_to_Tool_Changer_m.STL"/>
+                    <mesh filename="package://hpp-ipa/meshes/Tools_to_Tool_Changer_m.STL"/>
                 </geometry>
             </collision>

File: urdf/tool_gripper.urdf.xacro (robot description, xacro)
@@ -17,5 +17,5 @@
                 <origin xyz="0 0 0" rpy="0 0 0" />
                 <geometry>
-                    <mesh filename="package://hpp-dlr-ipa/meshes/Tool_Gripper_Shell_m.STL"/>
+                    <mesh filename="package://hpp-ipa/meshes/Tool_Gripper_Shell_m.STL"/>
                 </geometry>
                 <material name="greyish">
@@ -26,5 +26,5 @@
                 <origin xyz="0 0 0" rpy="0 0 0" />
                 <geometry>
-                    <mesh filename="package://hpp-dlr-ipa/meshes/Tool_Gripper_Shell_m.STL"/>
+                    <mesh filename="package://hpp-ipa/meshes/Tool_Gripper_Shell_m.STL"/>
                 </geometry>
             </collision>

File: urdf/tool_screwdriver.urdf.xacro (robot description, xacro)
@@ -17,5 +17,5 @@
                 <origin xyz="0 0 0" rpy="0 0 0" />
                 <geometry>
-                    <mesh filename="package://hpp-dlr-ipa/meshes/Tools_Screwdriver_Shell_m.STL"/>
+                    <mesh filename="package://hpp-ipa/meshes/Tools_Screwdriver_Shell_m.STL"/>
                 </geometry>
                 <material name="greyish">
@@ -26,5 +26,5 @@
                 <origin xyz="0 0 0" rpy="0 0 0" />
                 <geometry>
-                    <mesh filename="package://hpp-dlr-ipa/meshes/Tools_Screwdriver_Shell_m.STL"/>
+                    <mesh filename="package://hpp-ipa/meshes/Tools_Screwdriver_Shell_m.STL"/>
                 </geometry>
             </collision>
